Commit message: add trajectory enerator and dataloader for gp

File: autorally_description/urdf/autoRallyPlatform.urdf.xacro (robot description, xacro)
@@ -43,7 +43,9 @@
   <xacro:property name="tire_dia" value="0.19"/>
   <!-- <xacro:property name="hex_hub_depth" value="0.0"/>  -->
-  <xacro:property name="front_tire_width" value="0.072644"/>
+  <!-- <xacro:property name="front_tire_width" value="0.072644"/> -->
+  <xacro:property name="front_tire_width" value="0.212644"/>
   <xacro:property name="front_wheel_mass" value="0.82"/>
-  <xacro:property name="rear_tire_width" value="0.0762"/>
+  <!-- <xacro:property name="rear_tire_width" value="0.0762"/> -->
+  <xacro:property name="rear_tire_width" value="0.212644"/>
   <xacro:property name="rear_wheel_mass" value="0.89"/>
   <!-- hex_hub_dist is the distance between left and right hex hubs when

Commit message: add gplogger

File: autorally_description/urdf/autoRallyPlatform.urdf.xacro (robot description, xacro)
@@ -24,5 +24,6 @@
   <!-- Degree-to-radian conversions -->
   <xacro:property name="degrees_45" value="0.785398163"/>
-  <xacro:property name="degrees_21" value="0.3665191429"/>
+  <!-- <xacro:property name="degrees_21" value="0.3665191429"/> -->
+  <xacro:property name="degrees_25" value="0.4363"/>
   <xacro:property name="degrees_90" value="1.57079633"/>
   <!-- chassis_length is measured along the x axis, chassis_width
@@ -271,5 +272,5 @@
       <!-- cant the front wheels to improve traction -->
       <axis xyz="0 ${-lr_reflect*0.09950372}  0.99503719"/>
-      <limit lower="${-degrees_21}" upper="${degrees_21}"
+      <limit lower="${-degrees_25}" upper="${degrees_25}"
              effort="${servo_stall_torque}" velocity="${servo_no_load_speed}"/>
     </joint>
